Commit message: debug and add new tutorial for mapping

File: src/gazebo_environment/pepper_robot/pepper_description/urdf/pepper1.0_generated_urdf/pepperGazebo.xacro (robot description, xacro)
@@ -3,5 +3,5 @@
     <!-- MACROS FOR DISABLE LINKS -->
 	<xacro:property name="PI" value="3.14159265359" />
-    <xacro:macro name="DisabledLinks" params="side side_small">
+    <!-- <xacro:macro name="DisabledLinks" params="side side_small">
         <plugin name="${side}Finger11_link" filename="libroboticsgroup_gazebo_disable_link_plugin.so">
             <link>${side}Finger11_link</link>
@@ -49,8 +49,8 @@
             <link>${side_small}_gripper</link>
         </plugin>
-    </xacro:macro>
+    </xacro:macro>  -->
     <!-- MACROS FOR MIMIC JOINTS -->
     <!-- Fingers -->
-     <xacro:macro name="FingerMimics" params="side num">
+ <!--    <xacro:macro name="FingerMimics" params="side num">
         <plugin name="mimic_${side}Finger${num}1" filename="libroboticsgroup_gazebo_mimic_joint_plugin.so">
             <joint>${side}Hand</joint>
@@ -85,5 +85,5 @@
             <offset>${PI/4}</offset>
         </plugin>
-    </xacro:macro>
+    </xacro:macro> -->
     <!-- GAZEBO ROS CONTROL -->
     <gazebo>
@@ -93,5 +93,5 @@
             <robotSimType>gazebo_ros_control/DefaultRobotHWSim</robotSimType>
         </plugin>
-         <xacro:FingerMimics side="L" num="1"/>
+ <!--        <xacro:FingerMimics side="L" num="1"/>
         <xacro:FingerMimics side="L" num="2"/>
         <xacro:FingerMimics side="L" num="3"/>
@@ -104,5 +104,5 @@
         <xacro:ThumbMimics side="R"/>
         <xacro:DisabledLinks side="L" side_small="l"/>
-        <xacro:DisabledLinks side="R" side_small="r"/>
+        <xacro:DisabledLinks side="R" side_small="r"/>  -->
     </gazebo>
     <!-- END OF GAZEBO ROS CONTROL PLUGIN -->
@@ -211,5 +211,5 @@
         <turnGravityOff>true</turnGravityOff>
     </gazebo>
-     <gazebo reference="LFinger11_link">
+<!--     <gazebo reference="LFinger11_link">
         <mu1>0.5</mu1>
         <mu2>0.5</mu2>
@@ -294,5 +294,5 @@
         <selfCollide>false</selfCollide>
         <turnGravityOff>true</turnGravityOff>
-    </gazebo>
+    </gazebo>  -->
     <gazebo reference="Hip">
         <mu1>0.5</mu1>

File: src/gazebo_environment/pepper_robot/pepper_description/urdf/pepper1.0_generated_urdf/pepper_robot_CPU.xacro (robot description, xacro)
@@ -10,5 +10,5 @@
 	<xacro:include filename="pepper_arms.xacro"/>
 	<xacro:include filename="pepper_sensors.xacro"/>
-	<xacro:include filename="pepper_fingers.xacro"/>
+	<!-- <xacro:include filename="pepper_fingers.xacro"/> -->
 	<xacro:include filename="pepper_wheels.xacro"/>
 	<xacro:include filename="pepperGazeboCPU.xacro"/>
